File: CArraigeFanBreakout.kicad_pcb (KiCad board)
At the start: 2 copper layers, 47 x 23.5 mm, 19 parts, among them J1 Conn_01x02_Male, J11 Conn_01x02, J11 Conn_01x02_Male, J12 Conn_01x02_Male, J13 Conn_01x02, J2 Conn_01x02, J3 Conn_01x02, J4 Conn_01x02, J5 Conn_01x02_Male, J6 1751248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

Commit message: Add files via upload
Parts:
- added D4: LED, LED_SMD:LED_0805_2012Metric_Pad1.15x1.40mm_HandSolder, F.Cu at (127.5, 61.9)
- added R4: R, Resistor_SMD:R_0603_1608Metric_Pad0.98x0.95mm_HandSolder, F.Cu at (127.4, 64.4)
- J11, J13, J2, J3, J4: footprint Connector_JST:JST_XH_B2B-XH-AM_1x02_P2.50mm_Vertical -> CArraigeFanBreakout:JST_XH_B2B-XH-AM_1x02_P2.50mm_Vertical_DJP
- J7: value Conn_01x02_Male -> 1751248; footprint Connector_PinHeader_2.54mm:PinHeader_1x02_P2.54mm_Vertical -> CArraigeFanBreakout:Phoenix_Contact-1751248-0-0-0
- moved J8 11.0 mm to (112.9, 72.7)
- moved J12 9.40 mm to (92.3, 73.8)
- moved R3 6.87 mm to (115.5, 72.6), turned to 270 degrees
- moved D1 6.77 mm to (127.3, 69.0)
- moved J13 4.10 mm to (92.5, 67.7), turned to 0 degrees
- moved D3 4.05 mm to (115.0, 68.7), turned to 270 degrees
- moved R2 3.97 mm to (127.2, 76.3), turned to 0 degrees
- moved J9 3.55 mm to (104.1, 79.8)
- moved R1 3.05 mm to (127.3, 71.6)
- moved J7 1.68 mm to (102.0, 70.2), turned to 0 degrees
- turned J6 to 180 degrees
Connections:
- J7 pad 1: -V_IN -> +V_IN
- J7 pad 2: +V_IN -> -V_IN
Routing:
- net -V_IN: track 18.1 -> 56.7 mm, vias 2 -> 0
- net +V_IN: track 16.1 -> 41.1 mm, vias 2 -> 0
- net -V_Probe: track 6.35 -> 27.9 mm, vias 2 -> 0
- net +3V3: track 6.35 -> 27.0 mm, vias 2 -> 0
- net Z_PROBE_CONN: track 6.35 -> 25.6 mm, vias 2 -> 0
- net -FAN1: track 58.5 -> 43.8 mm, vias 3 -> 0
- net -THERM: track 26.7 -> 12.2 mm, vias 2 -> 0
- net +THERM: track 17.0 -> 12.3 mm, vias 2 -> 0
- net Net-(D1-Pad2): track 6.35 -> 2.67 mm
- net Net-(D2-Pad2): track 6.35 -> 3.23 mm
- net -V_LED: track 20.0 -> 22.8 mm, vias 4 -> 0
- net Net-(D4-Pad2): track 0.00 -> 2.60 mm
- net +V_LED: track 18.3 -> 16.5 mm, vias 2 -> 0
- net +FAN1: track 50.6 -> 49.2 mm, vias 3 -> 0
- net Net-(D3-Pad2): track 2.75 -> 2.17 mm
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Other:
- board size 47 x 23.5 mm -> 47.4 x 23.5 mm
