File: CArraigeFanBreakout.sch (KiCad schematic (older format))
At the start: 19 parts, among them J1 Conn_01x02_Male, J10 Conn_01x02_Male, J11 Conn_01x02, J12 Conn_01x02_Male, J13 Conn_01x02, J2 Conn_01x02, J3 Conn_01x02, J4 Conn_01x02, J5 Conn_01x02_Male, J6 1751248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

Commit message: Add files via upload
Parts:
- removed J10, J7: Conn_01x02_Male, Connector_PinHeader_2.54mm:PinHeader_1x02_P2.54mm_Vertical, symbol Connector:Conn_01x02_Male
- added D4: LED, LED_SMD:LED_0805_2012Metric_Pad1.15x1.40mm_HandSolder, symbol Device:LED
- added J7: 1751248, CArraigeFanBreakout:Phoenix_Contact-1751248-0-0-0, symbol eec:1751248
- added R4: R, Resistor_SMD:R_0603_1608Metric_Pad0.98x0.95mm_HandSolder, symbol Device:R
- J11, J13, J2, J3, J4: footprint Connector_JST:JST_XH_B2B-XH-AM_1x02_P2.50mm_Vertical -> CArraigeFanBreakout:JST_XH_B2B-XH-AM_1x02_P2.50mm_Vertical_DJP
Connections:
- wire segments 55 -> 61
