File: 3DP_HotEnd_Breakout.sch (KiCad schematic (older format))
At the start: 20 parts, among them J1 Conn_01x02_Male, J11 Conn_01x02, J12 Conn_01x02_Male, J13 Conn_01x02, J2 Conn_01x02, J3 Conn_01x02, J4 Conn_01x02, J5 Conn_01x02_Male, J6 1751248, J7 1751248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

Commit message: REV1
Parts:
- added H1, H2, H3, H4: MountingHole, MountingHole:MountingHole_3.2mm_M3, symbol Mechanical:MountingHole
- added J10, J14, J15: Conn_01x02_Male, Connector_PinHeader_2.54mm:PinHeader_1x02_P2.54mm_Vertical, symbol Connector:Conn_01x02_Male
- D1, D2, D3, D4: footprint LED_SMD:LED_0805_2012Metric_Pad1.15x1.40mm_HandSolder -> 3DP_HotEnd_Breakout:LED_0805_2012Metric_Pad1.15x1.40mm_HandSolder
- J11, J13, J2, J3, J4: footprint CArraigeFanBreakout:JST_XH_B2B-XH-AM_1x02_P2.50mm_Vertical_DJP -> 3DP_HotEnd_Breakout:JST_XH_B2B-XH-AM_1x02_P2.50mm_Vertical_DJP
- J6, J7: footprint CArraigeFanBreakout:Phoenix_Contact-1751248-0-0-0 -> 3DP_HotEnd_Breakout:Phoenix_Contact-1751248-0-0-0
Other:
- moved on the sheet: D1, D4, J12, J13, J6, J7, J8, J9, R1, R3, R4

Commit message: revised SMT pads
Parts:
- D1, D2, D3, D4: footprint 3DP_HotEnd_Breakout:LED_0805_2012Metric_Pad1.15x1.40mm_HandSolder -> 3DP_HotEnd_Breakout:LED_1206_3216Metric_Pad1.42x1.75mm_HandSolder
- R1, R2, R3, R4: footprint Resistor_SMD:R_0603_1608Metric_Pad0.98x0.95mm_HandSolder -> Resistor_SMD:R_1206_3216Metric_Pad1.30x1.75mm_HandSolder
Changed lines of the file:
@@
 F 0 "D1" H 1393 2067 50  0000 C CNN
 F 1 "LED" H 1393 1976 50  0000 C CNN
-F 2 "3DP_HotEnd_Breakout:LED_0805_2012Metric_Pad1.15x1.40mm_HandSolder" H 1400 1850 50  0001 C CNN
+F 2 "3DP_HotEnd_Breakout:LED_1206_3216Metric_Pad1.42x1.75mm_HandSolder" H 1400 1850 50  0001 C CNN
 F 3 "~" H 1400 1850 50  0001 C CNN
 	1    1400 1850
@@
 F 0 "R1" V 1493 1850 50  0000 C CNN
 F 1 "R" V 1584 1850 50  0000 C CNN
-F 2 "Resistor_SMD:R_0603_1608Metric_Pad0.98x0.95mm_HandSolder" V 1630 1850 50  0001 C CNN
+F 2 "Resistor_SMD:R_1206_3216Metric_Pad1.30x1.75mm_HandSolder" V 1630 1850 50  0001 C CNN
 F 3 "~" H 1700 1850 50  0001 C CNN
 	1    1700 1850
@@
 F 0 "D2" H 4300 1650 50  0000 C CNN
 F 1 "LED" H 4300 1800 50  0000 C TNN
-F 2 "3DP_HotEnd_Breakout:LED_0805_2012Metric_Pad1.15x1.40mm_HandSolder" H 4300 1850 50  0001 C CNN
+F 2 "3DP_HotEnd_Breakout:LED_1206_3216Metric_Pad1.42x1.75mm_HandSolder" H 4300 1850 50  0001 C CNN
 F 3 "~" H 4300 1850 50  0001 C CNN
 	1    4300 1850
@@
 F 0 "R2" V 4800 1850 50  0000 C CNN
 F 1 "R" V 4700 1850 50  0000 C CNN
-F 2 "Resistor_SMD:R_0603_1608Metric_Pad0.98x0.95mm_HandSolder" V 4530 1850 50  0001 C CNN
+F 2 "Resistor_SMD:R_1206_3216Metric_Pad1.30x1.75mm_HandSolder" V 4530 1850 50  0001 C CNN
 F 3 "~" H 4600 1850 50  0001 C CNN
 	1    4600 1850
@@
 F 0 "D3" H 1900 2850 50  0000 C CNN
 F 1 "LED" H 2100 2850 50  0000 C CNN
-F 2 "3DP_HotEnd_Breakout:LED_0805_2012Metric_Pad1.15x1.40mm_HandSolder" H 1900 2950 50  0001 C CNN
+F 2 "3DP_HotEnd_Breakout:LED_1206_3216Metric_Pad1.42x1.75mm_HandSolder" H 1900 2950 50  0001 C CNN
 F 3 "~" H 1900 2950 50  0001 C CNN
 	1    1900 2950
@@
 F 0 "R3" V 1550 3000 50  0000 L CNN
 F 1 "R" V 1550 2850 50  0000 L CNN
-F 2 "Resistor_SMD:R_0603_1608Metric_Pad0.98x0.95mm_HandSolder" V 1580 2950 50  0001 C CNN
+F 2 "Resistor_SMD:R_1206_3216Metric_Pad1.30x1.75mm_HandSolder" V 1580 2950 50  0001 C CNN
 F 3 "~" H 1650 2950 50  0001 C CNN
 	1    1650 2950
@@
 F 0 "D4" V 5789 1232 50  0000 R CNN
 F 1 "LED" V 5698 1232 50  0000 R CNN
-F 2 "3DP_HotEnd_Breakout:LED_0805_2012Metric_Pad1.15x1.40mm_HandSolder" H 5750 1350 50  0001 C CNN
+F 2 "3DP_HotEnd_Breakout:LED_1206_3216Metric_Pad1.42x1.75mm_HandSolder" H 5750 1350 50  0001 C CNN
 F 3 "~" H 5750 1350 50  0001 C CNN
 	1    5750 1350
@@
 F 0 "R4" H 5400 1400 50  0000 L CNN
 F 1 "R" H 5450 1300 50  0000 L CNN
-F 2 "Resistor_SMD:R_0603_1608Metric_Pad0.98x0.95mm_HandSolder" V 5530 1350 50  0001 C CNN
+F 2 "Resistor_SMD:R_1206_3216Metric_Pad1.30x1.75mm_HandSolder" V 5530 1350 50  0001 C CNN
 F 3 "~" H 5600 1350 50  0001 C CNN
 	1    5600 1350
